File: PCB/projects/BBB ledscape/GTOledscapeV0.4.sch (EAGLE design)
At the start: 16 parts

Commit message: PCB updated to use the 74AHCT245 chip instead of the other level shifter. Should work better for going from 3v3 to 5v
Parts:
- removed 74LVC245AN, 74LVC245AN1: (no value), tgo_custom:74LVC245
- removed C4: (no value), rcl:C-EU050-045X075
- removed CON3: (no value), con-harting:CON16
- removed R18: (no value), rcl:R-EU_0204/5
- removed U$1: BEAGLEBONE_OUTLINE, adafruit:BEAGLEBONE_OUTLINE
- added CON1: (no value), con-harting:CON16
- added IC1, IC2: 74HC245N, 74xx-eu:74HC245N
- added R1: (no value), rcl:R-EU_0204/5
- added U1: BEAGLEBONE_OUTLINE, adafruit:BEAGLEBONE_OUTLINE
- C1: device rcl:CPOL-EUE2.5-7 -> rcl:C-EU050-045X075
- C3: device rcl:C-EU050-045X075 -> rcl:CPOL-EUE2.5-7
- renumbered R17 to R2
Connections:
- removed net N$21: 74LVC245AN1.B1, RN2A.1
- removed net N$22: 74LVC245AN1.B2, RN2B.1
- removed net N$23: 74LVC245AN1.B3, RN2C.1
- removed net N$24: 74LVC245AN1.B4, RN2D.1
- removed net N$25: 74LVC245AN1.B5, RN2E.1
- removed net N$26: 74LVC245AN1.B6, RN2F.1
- removed net N$27: 74LVC245AN1.B7, RN2G.1
- removed net N$28: 74LVC245AN1.B8, RN2H.1
- removed net VDD_V3V: 74LVC245AN.VCC, 74LVC245AN1.VCC
- new net N$10: IC1A.B2, RN1B.1
- new net N$11: IC1A.B3, RN1C.1
- new net N$12: IC1A.B4, RN1D.1
- new net N$13: IC1A.B5, RN1E.1
- new net N$14: IC1A.B6, RN1F.1
- new net N$29: IC1A.B7, RN1G.1
- new net N$30: IC1A.B8, RN1H.1
- new net N$7: IC1A.B1, RN1A.1
- net +5V: now also C1.1, C3.+, IC1A.DIR, IC1P.VCC, IC2A.DIR, IC2P.VCC, LED2.A, U1.SYS_5V@1, U1.SYS_5V@2; no longer C1.+, C3.1, C4.1, LED1.A
- net CH00: now also IC1A.A1, U1.UART5_RTSN; no longer 74LVC245AN1.A1, U$1.UART5_RTSN
- net CH00_OP: now also CON1.1, RN1A.2; no longer CON3.1, RN2A.2
- net CH01: now also IC1A.A2, U1.GPIO2_25; no longer 74LVC245AN1.A2, U$1.GPIO2_25
- net CH01_OP: now also CON1.3, RN1B.2; no longer CON3.3, RN2B.2
- net CH02: now also IC1A.A3, U1.GPIO2_1; no longer 74LVC245AN1.A3, U$1.GPIO2_1
- net CH02_OP: now also CON1.5, RN1C.2; no longer CON3.5, RN2C.2
- net CH03: now also IC1A.A4, U1.GPIO1_14; no longer 74LVC245AN1.A4, U$1.GPIO1_14
- net CH03_OP: now also CON1.7, RN1D.2; no longer CON3.7, RN2D.2
- net CH04: now also IC1A.A5, U1.GPIO0_26; no longer 74LVC245AN1.A5, U$1.GPIO0_26
- net CH04_OP: now also CON1.9, RN1E.2; no longer CON3.9, RN2E.2
- net CH05: now also IC1A.A6, U1.GPIO1_12; no longer 74LVC245AN1.A6, U$1.GPIO1_12
- net CH05_OP: now also CON1.11, RN1F.2; no longer CON3.11, RN2F.2
- net CH06: now also IC1A.A7, U1.TIMER6; no longer 74LVC245AN1.A7, U$1.TIMER6
- net CH06_OP: now also CON1.13, RN1G.2; no longer CON3.13, RN2G.2
- net CH07: now also IC1A.A8, U1.TIMER7; no longer 74LVC245AN1.A8, U$1.TIMER7
- net CH07_OP: now also CON1.15, RN1H.2; no longer CON3.15, RN2H.2
- net CH08: now also IC2A.A1, U1.GPIO2_6; no longer 74LVC245AN.A1, U$1.GPIO2_6
- net CH08_OP: now also RN2A.2; no longer RN1A.2
- net CH09: now also IC2A.A2, U1.GPIO2_7; no longer 74LVC245AN.A2, U$1.GPIO2_7
- net CH09_OP: now also RN2B.2; no longer RN1B.2
- net CH10: now also IC2A.A3, U1.GPIO2_9; no longer 74LVC245AN.A3, U$1.GPIO2_9
- net CH10_OP: now also RN2C.2; no longer RN1C.2
- net CH11: now also IC2A.A4, U1.GPIO2_11; no longer 74LVC245AN.A4, U$1.GPIO2_11
- net CH11_OP: now also RN2D.2; no longer RN1D.2
- net CH12: now also IC2A.A5, U1.GPIO2_13; no longer 74LVC245AN.A5, U$1.GPIO2_13
- net CH12_OP: now also RN2E.2; no longer RN1E.2
- net CH13: now also IC2A.A6, U1.UART5_RXD; no longer 74LVC245AN.A6, U$1.UART5_RXD
- net CH13_OP: now also RN2F.2; no longer RN1F.2
- net CH14: now also IC2A.A7, U1.UART3_CTSN; no longer 74LVC245AN.A7, U$1.UART3_CTSN
- net CH14_OP: now also RN2G.2; no longer RN1G.2
- net CH15: now also IC2A.A8, U1.UART3_RTSN; no longer 74LVC245AN.A8, U$1.UART3_RTSN
- net CH15_OP: now also RN2H.2; no longer RN1H.2
- net GND: now also C1.2, C3.-, CON1.10, CON1.12, CON1.14, CON1.16, CON1.2, CON1.4, CON1.6, CON1.8, IC1A.G, IC1P.GND, IC2A.G, IC2P.GND, R1.1, U1.GND@1, U1.GND@2, U1.GND@3, U1.GND@4, U1.GND@5, U1.GND@6, U1.GND@7, U1.GND@8; no longer 74LVC245AN.GND, 74LVC245AN.OE, 74LVC245AN1.GND, 74LVC245AN1.OE, C1.-, C3.2, C4.2, CON3.10, CON3.12, CON3.14, CON3.16, CON3.2, CON3.4, CON3.6, CON3.8, R18.1, U$1.GND@7, U$1.GND@8
- net N$1: now also IC2A.B1, RN2A.1; no longer 74LVC245AN.B1, RN1A.1
- net N$15: now also IC2A.B3, RN2C.1; no longer 74LVC245AN.B3, RN1C.1
- net N$16: now also IC2A.B4, RN2D.1; no longer 74LVC245AN.B4, RN1D.1
- net N$17: now also IC2A.B5, RN2E.1; no longer 74LVC245AN.B5, RN1E.1
- net N$18: now also IC2A.B6, RN2F.1; no longer 74LVC245AN.B6, RN1F.1
- net N$19: now also IC2A.B7, RN2G.1; no longer 74LVC245AN.B7, RN1G.1
- net N$2: now also LED2.C; no longer LED1.C
- net N$20: now also IC2A.B8, RN2H.1; no longer 74LVC245AN.B8, RN1H.1
- net N$3: now also LED1.C, R1.2; no longer LED2.C, R18.2
- net N$4: now also LED1.A, U1.GPIO1_17; no longer LED2.A, U$1.GPIO1_17
- net N$6: now also IC2A.B2, RN2B.1; no longer 74LVC245AN.B2, RN1B.1
- net UART1_RXD: now also U1.UART1_RXD; no longer U$1.UART1_RXD
- net UART1_TXD: now also U1.UART1_TXD; no longer U$1.UART1_TXD
- net VDD_3V3: now also U1.VDD_3V3EXP@1; no longer 74LVC245AN.DIR, 74LVC245AN1.DIR, U$1.VDD_3V3EXP@1
Other:
- note added: "Ben Holden"
- moved on the sheet: C2, CON2, LED1, LED2, RN1A, RN1B, RN1C, RN1D, RN1E, RN1F, RN1G, RN1H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
